File: Nanino8/Nanino8.kicad_pcb (KiCad board)
At the start: 2 copper layers, 68.6 x 53.3 mm, 63 parts, among them IC1 ATMEGA328-P, P1 POWER, P2 ANALOG, P3 SERIAL, P4 DIGITAL 0-7, P5 DIGITAL 8-13, P6 3V3, P7 VIN, SW1 SW_PUSH, X1 16 MHz

Commit message: Generated gerbers
Parts:
- removed the ? at (102.9, 105.4)
- removed the ? at (108.0, 113.0)
- removed the ? at (110.5, 113.0)
- removed the ? at (113.0, 113.0)
- removed the ? at (115.6, 113.0)
- removed the ? at (105.4, 105.4)
- removed the ? at (113.0, 105.4)
- removed the ? at (115.6, 105.4)
- removed the ? at (102.9, 92.7)
- removed the ? at (105.4, 92.7)
- removed the ? at (108.0, 92.7)
- removed the ? at (110.5, 92.7)
- removed the ? at (113.0, 92.7)
- removed the ? at (115.6, 92.7)
- removed the ? at (102.9, 85.1)
- removed the ? at (105.4, 85.1)
- removed the ? at (108.0, 85.1)
- removed the ? at (110.5, 85.1)
- removed the ? at (113.0, 85.1)
- removed the ? at (115.6, 85.1)
- removed the ? at (102.9, 77.5)
- removed the ? at (113.0, 77.5)
- removed the ? at (105.4, 113.0)
- removed the ? at (108.0, 77.5)
- removed the ? at (110.5, 105.4)
- removed the ? at (102.9, 113.0)
- removed the ? at (108.0, 105.4)
- removed the ? at (102.9, 120.7)
- removed the ? at (105.4, 77.5)
- removed the ? at (110.5, 77.5)
- removed the ? at (115.6, 77.5)
- removed the ? at (105.4, 120.7)
- removed the ? at (108.0, 120.7)
- removed the ? at (110.5, 120.7)
- removed the ? at (113.0, 120.7)
- removed the ? at (115.6, 120.7)
- added ?: , a-dh-libmod:Proto-3, F.Cu at (115.6, 125.7)
- added ?: , a-dh-libmod:Proto-3, F.Cu at (108.0, 118.1)
- added ?: , a-dh-libmod:Proto-3, F.Cu at (105.4, 118.1)
- added ?: , a-dh-libmod:Proto-3, F.Cu at (102.9, 118.1)
- added ?: , a-dh-libmod:Proto-3, F.Cu at (115.6, 110.5)
- added ?: , a-dh-libmod:Proto-3, F.Cu at (113.0, 110.5)
- added ?: , a-dh-libmod:Proto-3, F.Cu at (110.5, 110.5)
- added ?: , a-dh-libmod:Proto-3, F.Cu at (108.0, 110.5)
- added ?: , a-dh-libmod:Proto-3, F.Cu at (105.4, 110.5)
- added ?: , a-dh-libmod:Proto-3, F.Cu at (102.9, 110.5)
- added ?: , a-dh-libmod:Proto-3, F.Cu at (115.6, 97.8)
- added ?: , a-dh-libmod:Proto-3, F.Cu at (113.0, 125.7)
- added ?: , a-dh-libmod:Proto-3, F.Cu at (113.0, 97.8)
- added ?: , a-dh-libmod:Proto-3, F.Cu at (110.5, 97.8)
- added ?: , a-dh-libmod:Proto-3, F.Cu at (108.0, 97.8)
- added ?: , a-dh-libmod:Proto-3, F.Cu at (105.4, 97.8)
- added ?: , a-dh-libmod:Proto-3, F.Cu at (102.9, 97.8)
- added ?: , a-dh-libmod:Proto-3, F.Cu at (115.6, 90.2)
- added ?: , a-dh-libmod:Proto-3, F.Cu at (113.0, 90.2)
- added ?: , a-dh-libmod:Proto-3, F.Cu at (110.5, 90.2)
- added ?: , a-dh-libmod:Proto-3, F.Cu at (108.0, 90.2)
- added ?: , a-dh-libmod:Proto-3, F.Cu at (105.4, 90.2)
- added ?: , a-dh-libmod:Proto-3, F.Cu at (110.5, 125.7)
- added ?: , a-dh-libmod:Proto-3, F.Cu at (102.9, 90.2)
- added ?: , a-dh-libmod:Proto-3, F.Cu at (115.6, 82.5)
- added ?: , a-dh-libmod:Proto-3, F.Cu at (113.0, 82.5)
- added ?: , a-dh-libmod:Proto-3, F.Cu at (110.5, 82.5)
- added ?: , a-dh-libmod:Proto-3, F.Cu at (108.0, 82.5)
- added ?: , a-dh-libmod:Proto-3, F.Cu at (105.4, 82.5)
- added ?: , a-dh-libmod:Proto-3, F.Cu at (108.0, 125.7)
- added ?: , a-dh-libmod:Proto-3, F.Cu at (102.9, 82.5)
- added ?: , a-dh-libmod:Proto-3, F.Cu at (105.4, 125.7)
- added ?: , a-dh-libmod:Proto-3, F.Cu at (102.9, 125.7)
- added ?: , a-dh-libmod:Proto-3, F.Cu at (115.6, 118.1)
- added ?: , a-dh-libmod:Proto-3, F.Cu at (113.0, 118.1)
- added ?: , a-dh-libmod:Proto-3, F.Cu at (110.5, 118.1)
- renumbered P6 to ?
Routing:
- net Net-(P32-Pad1): track 8.24 -> 0.00 mm
- net Net-(P35-Pad1): track 8.06 -> 0.00 mm
- net Net-(P21-Pad1): track 8.06 -> 0.00 mm
- net Net-(P41-Pad1): track 8.06 -> 0.00 mm
- net Net-(P39-Pad1): track 8.06 -> 0.00 mm
- net Net-(P29-Pad1): track 8.06 -> 0.00 mm
- net Net-(P23-Pad1): track 8.06 -> 0.00 mm
- net Net-(P49-Pad1): track 8.06 -> 0.00 mm
- net Net-(P43-Pad1): track 8.06 -> 0.00 mm
- net Net-(P13-Pad1): track 8.06 -> 0.00 mm
- net Net-(P38-Pad1): track 7.88 -> 0.00 mm
- net Net-(P34-Pad1): track 7.62 -> 0.00 mm
- net Net-(P33-Pad1): track 7.62 -> 0.00 mm
- net Net-(P31-Pad1): track 7.62 -> 0.00 mm
- net Net-(P30-Pad1): track 7.62 -> 0.00 mm
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
Commit message: Updated for Course Session 1
Parts:
- removed the ? at (115.6, 125.7)
- removed the ? at (108.0, 118.1)
- removed the ? at (105.4, 118.1)
- removed the ? at (102.9, 118.1)
- removed the ? at (115.6, 110.5)
- removed the ? at (113.0, 110.5)
- removed the ? at (110.5, 110.5)
- removed the ? at (108.0, 110.5)
- removed the ? at (105.4, 110.5)
- removed the ? at (102.9, 110.5)
- removed the ? at (115.6, 97.8)
- removed the ? at (113.0, 125.7)
- removed the ? at (113.0, 97.8)
- removed the ? at (110.5, 97.8)
- removed the ? at (108.0, 97.8)
- removed the ? at (105.4, 97.8)
- removed the ? at (102.9, 97.8)
- removed the ? at (115.6, 90.2)
- removed the ? at (113.0, 90.2)
- removed the ? at (110.5, 90.2)
- removed the ? at (108.0, 90.2)
- removed the ? at (105.4, 90.2)
- removed the ? at (110.5, 125.7)
- removed the ? at (102.9, 90.2)
- removed the ? at (115.6, 82.5)
- removed the ? at (113.0, 82.5)
- removed the ? at (110.5, 82.5)
- removed the ? at (108.0, 82.5)
- removed the ? at (105.4, 82.5)
- removed the ? at (108.0, 125.7)
- removed the ? at (102.9, 82.5)
- removed the ? at (105.4, 125.7)
- removed the ? at (102.9, 125.7)
- removed the ? at (115.6, 118.1)
- removed the ? at (113.0, 118.1)
- removed the ? at (110.5, 118.1)
- added Ref**11: Val**, a-dh-libmod:Proto-3, F.Cu at (102.9, 110.5)
- added Ref**111: Val**, a-dh-libmod:Proto-3, F.Cu at (102.9, 82.5)
- added Ref**112: Val**, a-dh-libmod:Proto-3, F.Cu at (102.9, 90.2)
- added Ref**113: Val**, a-dh-libmod:Proto-3, F.Cu at (102.9, 97.8)
- added Ref**12: Val**, a-dh-libmod:Proto-3, F.Cu at (102.9, 118.1)
- added Ref**121: Val**, a-dh-libmod:Proto-3, F.Cu at (105.4, 82.5)
- added Ref**122: Val**, a-dh-libmod:Proto-3, F.Cu at (105.4, 90.2)
- added Ref**123: Val**, a-dh-libmod:Proto-3, F.Cu at (105.4, 97.8)
- added Ref**13: Val**, a-dh-libmod:Proto-3, F.Cu at (102.9, 125.7)
- added Ref**131: Val**, a-dh-libmod:Proto-3, F.Cu at (108.0, 82.5)
- added Ref**132: Val**, a-dh-libmod:Proto-3, F.Cu at (108.0, 90.2)
- added Ref**133: Val**, a-dh-libmod:Proto-3, F.Cu at (108.0, 97.8)
- added Ref**141: Val**, a-dh-libmod:Proto-3, F.Cu at (110.5, 82.5)
- added Ref**142: Val**, a-dh-libmod:Proto-3, F.Cu at (110.5, 90.2)
- added Ref**143: Val**, a-dh-libmod:Proto-3, F.Cu at (110.5, 97.8)
- added Ref**151: Val**, a-dh-libmod:Proto-3, F.Cu at (113.0, 82.5)
- added Ref**152: Val**, a-dh-libmod:Proto-3, F.Cu at (113.0, 90.2)
- added Ref**153: Val**, a-dh-libmod:Proto-3, F.Cu at (113.0, 97.8)
- added Ref**161: Val**, a-dh-libmod:Proto-3, F.Cu at (115.6, 82.5)
- added Ref**162: Val**, a-dh-libmod:Proto-3, F.Cu at (115.6, 90.2)
- added Ref**163: Val**, a-dh-libmod:Proto-3, F.Cu at (115.6, 97.8)
- added Ref**21: Val**, a-dh-libmod:Proto-3, F.Cu at (105.4, 110.5)
- added Ref**22: Val**, a-dh-libmod:Proto-3, F.Cu at (105.4, 118.1)
- added Ref**23: Val**, a-dh-libmod:Proto-3, F.Cu at (105.4, 125.7)
- added Ref**31: Val**, a-dh-libmod:Proto-3, F.Cu at (108.0, 110.5)
- added Ref**32: Val**, a-dh-libmod:Proto-3, F.Cu at (108.0, 118.1)
- added Ref**33: Val**, a-dh-libmod:Proto-3, F.Cu at (108.0, 125.7)
- added Ref**41: Val**, a-dh-libmod:Proto-3, F.Cu at (110.5, 110.5)
- added Ref**42: Val**, a-dh-libmod:Proto-3, F.Cu at (110.5, 118.1)
- added Ref**43: Val**, a-dh-libmod:Proto-3, F.Cu at (110.5, 125.7)
- added Ref**51: Val**, a-dh-libmod:Proto-3, F.Cu at (113.0, 110.5)
- added Ref**52: Val**, a-dh-libmod:Proto-3, F.Cu at (113.0, 118.1)
- added Ref**53: Val**, a-dh-libmod:Proto-3, F.Cu at (113.0, 125.7)
- added Ref**61: Val**, a-dh-libmod:Proto-3, F.Cu at (115.6, 110.5)
- added Ref**62: Val**, a-dh-libmod:Proto-3, F.Cu at (115.6, 118.1)
- added Ref**63: Val**, a-dh-libmod:Proto-3, F.Cu at (115.6, 125.7)
- C1, C3, C4: footprint Capacitors_ThroughHole:C_Rect_L4_W2.5_P2.5 -> a-dh-libmod:C_Rect_L4_W2.5_P2.5_Mill
- moved P7 0.38 mm to (143.5, 122.8)
- moved C4 0.18 mm to (136.7, 105.9)
- gave numbers to parts that had none: 7
Routing:
- net GND: track 259.3 -> 225.1 mm
- net VCC: track 206.8 -> 178.1 mm
- net /A4: track 20.3 -> 18.6 mm
- net AREF: track 43.2 -> 44.1 mm
- net RESET: track 67.3 -> 66.4 mm
Other:
- net class Default: clearance 0.2 -> 0.4826
- net class Proto: clearance 0.2 -> 0.4826
- rule trace_clearance: 0.2 -> 0.4826
- rule trace_min: 0.8128 -> 0.8
