File: Nanino8/Nanino8.sch (KiCad schematic (older format))
At the start: 61 parts, among them IC1 ATMEGA328-P, P1 POWER, P12 CONN_01X03, P13 CONN_01X03, P14 CONN_01X03, P15 CONN_01X03, P16 CONN_01X03, P17 CONN_01X03, P18 CONN_01X06, P19 CONN_01X10, P2 ANALOG, P20 CONN_01X03, P21 CONN_01X03, P22 CONN_01X03, P23 CONN_01X03, P24 CONN_01X03, P25 CONN_01X03, P26 CONN_01X06, P27 CONN_01X10, P28 CONN_01X03, P29 CONN_01X03, P3 SERIAL, P30 CONN_01X03, P31 CONN_01X03, P32 CONN_01X03, P33 CONN_01X03, P34 CONN_01X03, P35 CONN_01X03, P36 CONN_01X03, P37 CONN_01X03, P38 CONN_01X03, P39 CONN_01X03, P4 DIGITAL 0-7, P40 CONN_01X03, P41 CONN_01X03, P42 CONN_01X03, P43 CONN_01X03, P44 CONN_01X03, P45 CONN_01X03, P46 CONN_01X03, P47 CONN_01X03, P48 CONN_01X03, P49 CONN_01X03, P5 DIGITAL 8-13, P50 CONN_01X03, P51 CONN_01X03, P6 3V3, P7 VIN, P8 CONN_01X02, P9 CONN_01X02, SW1 SW_PUSH, X1 16 MHz

Commit message: Generated gerbers
Parts:
- removed P12, P13, P14, P15, P16, P17, P20, P21, P22, P23, P24, P25, P28, P29, P30, P31, P32, P33, P34, P35, P36, P37, P38, P39, P40, P41, P42, P43, P44, P45, P46, P47, P48, P49, P50, P51: CONN_01X03, Pin_Headers:Pin_Header_Straight_1x03, symbol CONN_01X03

Commit message: Updated for Course Session 1
Parts:
- C1, C3, C4: footprint Capacitors_ThroughHole:C_Rect_L4_W2.5_P2.5 -> a-dh-libmod:C_Rect_L4_W2.5_P2.5_Mill
Changed lines of the file:
@@
 F 0 "IC1" H 5150 4650 50  0000 L BNN
 F 1 "ATMEGA328-P" H 5750 2000 50  0000 L BNN
-F 2 "Housings_DIP:DIP-28_W7.62mm_LongPads" H 5900 3400 50  0000 C CIN
+F 2 "Housings_DIP:DIP-28_W7.62mm_LongPads" V 5600 3450 50  0000 C CIN
 F 3 "" H 5900 3400 50  0000 C CNN
 	1    5900 3400
@@
 F 0 "C3" H 6175 1350 50  0000 L CNN
 F 1 "0.1uF" H 6175 1150 50  0000 L CNN
-F 2 "Capacitors_ThroughHole:C_Rect_L4_W2.5_P2.5" H 6188 1100 50  0001 C CNN
+F 2 "a-dh-libmod:C_Rect_L4_W2.5_P2.5_Mill" H 6188 1100 50  0001 C CNN
 F 3 "" H 6150 1250 50  0000 C CNN
 	1    6150 1250
@@
 F 0 "C1" H 3775 3100 50  0000 L CNN
 F 1 "0.1uF" H 3775 2900 50  0000 L CNN
-F 2 "Capacitors_ThroughHole:C_Rect_L4_W2.5_P2.5" H 3788 2850 50  0001 C CNN
+F 2 "a-dh-libmod:C_Rect_L4_W2.5_P2.5_Mill" H 3788 2850 50  0001 C CNN
 F 3 "" H 3750 3000 50  0000 C CNN
 	1    3750 3000
@@
 F 0 "C4" H 4775 3350 50  0000 L CNN
 F 1 "0.1uF" H 4775 3150 50  0000 L CNN
-F 2 "Capacitors_ThroughHole:C_Rect_L4_W2.5_P2.5" H 4788 3100 50  0001 C CNN
+F 2 "a-dh-libmod:C_Rect_L4_W2.5_P2.5_Mill" H 4788 3100 50  0001 C CNN
 F 3 "" H 4750 3250 50  0000 C CNN
 	1    4750 3250
