File: Test/Test.sch (KiCad schematic (older format))
At the start: 5 parts, among them P1 CONN_01X02, P2 CONN_01X03, SW1 SW_PUSH

Commit message: Updated for Course Session 1
Parts:
- removed X?: CER_RESO, symbol CER_RESO
Changed lines of the file:
@@
 P 3150 3250
 F 0 "P1" H 3150 3400 50  0000 C CNN
-F 1 "CONN_01X02" V 3250 3250 50  0000 C CNN
+F 1 "CONN_01X02" V 3250 3250 50  0001 C CNN
 F 2 "Pin_Headers:Pin_Header_Straight_1x02" H 3150 3250 50  0001 C CNN
 F 3 "" H 3150 3250 50  0000 C CNN
@@
 P 4950 3200
 F 0 "P2" H 4950 3400 50  0000 C CNN
-F 1 "CONN_01X03" V 5050 3200 50  0000 C CNN
+F 1 "CONN_01X03" V 5050 3200 50  0001 C CNN
 F 2 "Pin_Headers:Pin_Header_Straight_1x03" H 4950 3200 50  0001 C CNN
 F 3 "" H 4950 3200 50  0000 C CNN
@@
 Wire Wire Line
 	3350 3200 4750 3200
-Text Label 3600 3300 0    60   ~ 0
-GND
-Text Label 3600 3200 0    60   ~ 0
-VCC
 Wire Wire Line
 	3850 3000 3850 3300
@@
 	1    0    0    -1
 $EndComp
+Text Label 4650 3100 0    60   ~ 0
+SW
+Text Label 3600 3200 0    60   ~ 0
+VCC
+Text Label 3600 3300 0    60   ~ 0
+GND
 $Comp
 L PWR_FLAG #FLG02
-U 1 1 57A6DC65
+U 1 1 57B55A25
 P 3400 3100
 F 0 "#FLG02" H 3400 3195 50  0001 C CNN
@@
 $Comp
 L PWR_FLAG #FLG03
-U 1 1 57A6DCE5
+U 1 1 57B55A45
 P 3400 3400
 F 0 "#FLG03" H 3400 3495 50  0001 C CNN
@@
 	3400 3400 3400 3300
 Connection ~ 3400 3300
-Text Label 4650 3100 0    60   ~ 0
-SW
-$Comp
-L CER_RESO X?
-U 1 1 57A77A74
-P 3850 1850
-F 0 "X?" H 3850 2000 60  0000 C CNN
-F 1 "CER_RESO" H 3850 2100 60  0000 C CNN
-F 2 "" H 3850 1850 60  0000 C CNN
-F 3 "" H 3850 1850 60  0000 C CNN
-	1    3850 1850
-	1    0    0    -1
-$EndComp
 $EndSCHEMATC
